File: EE/servo-control-module/servo-control-module.kicad_pcb (KiCad board)
At the start: 2 copper layers, 4 parts, among them J1 SERVO, J2 USB, U1 ATtiny85-20P

Commit message: Updates for first milled board.
Parts:
- J1: footprint Connector_PinHeader_1.27mm:PinHeader_1x03_P1.27mm_Vertical -> Connector_PinHeader_2.54mm:PinHeader_1x03_P2.54mm_Vertical
- J2: footprint Connector_PinHeader_1.27mm:PinHeader_1x05_P1.27mm_Vertical -> Connector_PinSocket_2.54mm:PinSocket_1x05_P2.54mm_Vertical
- RV1: footprint Potentiometer_THT:Potentiometer_Vishay_148-149_Single_Horizontal -> Potentiometer_THT:Potentiometer_Alps_RK163_Single_Horizontal
- moved RV1 20.9 mm to (105.9, 109.8), turned to 90 degrees
- moved J1 14.3 mm to (120.4, 90.2)
- moved U1 6.04 mm to (107.6, 90.2)
- moved J2 4.85 mm to (116.0, 84.2)
Connections:
- U1 pad 6: SERVO -> unconnected-(U1-PB1-Pad6)
- U1 pad 7: unconnected-(U1-PB2-Pad7) -> SERVO
Routing:
- net +5V: track 0.00 -> 43.7 mm
- net V-POT: track 0.00 -> 18.4 mm
- net SERVO: track 0.00 -> 5.06 mm
- added copper zone on B.Cu, net GND
Other:
- board outline added: 27.8 x 35.4 mm
